Commit message: started creating standalone kmp200 urdf

File: src/kmriiwa_description/urdf/iiwa14/iiwa14.xacro (robot description, xacro)
@@ -2,9 +2,9 @@
 <robot xmlns:xacro="http://www.ros.org/wiki/xacro">
   <!-- Import all Gazebo-customization elements, including Gazebo colors -->
-  <xacro:include filename="$(find kmriiwa_description)/urdf/iiwa14/iiwa.gazebo.xacro" />
+  <xacro:include filename="$(find kmriiwa_description)/urdf/lbriiwa14/iiwa.gazebo.xacro" />
   <!-- Import Transmissions -->
-  <xacro:include filename="$(find kmriiwa_description)/urdf/iiwa14/iiwa.transmission.xacro" />
+  <xacro:include filename="$(find kmriiwa_description)/urdf/lbriiwa14/iiwa.transmission.xacro" />
   <!-- Include Utilities -->
-  <xacro:include filename="$(find kmriiwa_description)/urdf/iiwa14/utilities.xacro" />
+  <xacro:include filename="$(find kmriiwa_description)/urdf/lbriiwa14/utilities.xacro" />
   <!-- some constants -->
   <xacro:property name="safety_controller_k_pos" value="100" />
@@ -13,11 +13,12 @@
   <xacro:property name="max_effort" value="300"/>
   <xacro:property name="max_velocity" value="10"/>
+  <xacro:property name="robot_name" value="iiwa14"/>
   <xacro:macro name="iiwa14" params="parent hardware_interface robot_name *origin">
     <!--joint between {parent} and link_0-->
-    <joint name="${parent}_${robot_name}_joint" type="fixed">
+    <!-- <joint name="${parent}_${robot_name}_joint" type="fixed">
       <xacro:insert_block name="origin"/>
       <parent link="${parent}"/>
       <child link="${robot_name}_link_0"/>
-    </joint>
+    </joint> -->
     <link name="${robot_name}_link_0">
       <inertial>

File: src/kmriiwa_description/urdf/kmp200/kmp200.xacro (robot description, xacro)
@@ -155,5 +155,5 @@
         </inertial> -->
     </link>
-    <joint name="${robot_name}_front_left_wheel_joint" type="fixed">
+    <joint name="${robot_name}_front_left_wheel_joint" type="revolute">
         <parent link="${robot_name}_base_link"/>
         <child link="${robot_name}_front_left_wheel_link"/>
@@ -163,5 +163,5 @@
         <joint_properties damping="0.0" friction="0.0"/>
     </joint>
-    <joint name="${robot_name}_front_right_wheel_joint" type="fixed">
+    <joint name="${robot_name}_front_right_wheel_joint" type="revolute">
         <parent link="${robot_name}_base_link"/>
         <child link="${robot_name}_front_right_wheel_link"/>
@@ -171,5 +171,5 @@
         <joint_properties damping="0.0" friction="0.0"/>
     </joint>
-    <joint name="${robot_name}_back_left_wheel_joint" type="fixed">
+    <joint name="${robot_name}_back_left_wheel_joint" type="revolute">
         <parent link="${robot_name}_base_link"/>
         <child link="${robot_name}_back_left_wheel_link"/>
@@ -179,5 +179,5 @@
         <joint_properties damping="0.0" friction="0.0"/>
     </joint>
-    <joint name="${robot_name}_back_right_wheel_joint" type="fixed">
+    <joint name="${robot_name}_back_right_wheel_joint" type="revolute">
         <parent link="${robot_name}_base_link"/>
         <child link="${robot_name}_back_right_wheel_link"/>

File: src/kmriiwa_description/urdf/robot/kmriiwa.urdf (robot description, URDF)
Before this commit: robot kmriiwa, 19 links, 18 joints
Joints:
- joint kmriiwa_back_left_wheel_joint: type fixed -> revolute
- joint kmriiwa_back_right_wheel_joint: type fixed -> revolute
- joint kmriiwa_front_left_wheel_joint: type fixed -> revolute
- joint kmriiwa_front_right_wheel_joint: type fixed -> revolute

Commit message: Created urdf without wheels and links

File: src/kmriiwa_description/urdf/iiwa14/iiwa14.xacro (robot description, xacro)
@@ -2,9 +2,9 @@
 <robot xmlns:xacro="http://www.ros.org/wiki/xacro">
   <!-- Import all Gazebo-customization elements, including Gazebo colors -->
-  <xacro:include filename="$(find kmriiwa_description)/urdf/lbriiwa14/iiwa.gazebo.xacro" />
+  <xacro:include filename="$(find kmriiwa_description)/urdf/iiwa14/iiwa.gazebo.xacro" />
   <!-- Import Transmissions -->
-  <xacro:include filename="$(find kmriiwa_description)/urdf/lbriiwa14/iiwa.transmission.xacro" />
+  <xacro:include filename="$(find kmriiwa_description)/urdf/iiwa14/iiwa.transmission.xacro" />
   <!-- Include Utilities -->
-  <xacro:include filename="$(find kmriiwa_description)/urdf/lbriiwa14/utilities.xacro" />
+  <xacro:include filename="$(find kmriiwa_description)/urdf/iiwa14/utilities.xacro" />
   <!-- some constants -->
   <xacro:property name="safety_controller_k_pos" value="100" />
@@ -16,9 +16,9 @@
   <xacro:macro name="iiwa14" params="parent hardware_interface robot_name *origin">
     <!--joint between {parent} and link_0-->
-    <!-- <joint name="${parent}_${robot_name}_joint" type="fixed">
+    <joint name="${parent}_${robot_name}_joint" type="fixed">
       <xacro:insert_block name="origin"/>
       <parent link="${parent}"/>
       <child link="${robot_name}_link_0"/>
-    </joint> -->
+    </joint>
     <link name="${robot_name}_link_0">
       <inertial>
